File: kicad/EPD_1in9/EPD_1in9.kicad_pcb (KiCad board)
At the start: 2 copper layers, 34 x 51 mm, 10 parts, among them J1 Conn_01x02, J2 Conn_01x08, J3 Conn_01x08, J4 Conn_01x08

Commit message: EPD_1in9: Add schematic symbol and footprint for the display outline
Parts:
- added Disp1: Waveshare_EPD_1in9, Display_local:Waveshare_EPD_1in9, F.Cu at (31.0, 80.2)
Other:
- board text added: "Chris Baker 2023"
Changed lines of the file:
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@@
   (net 17 "unconnected-(J3-Pad8)")
   (net 18 "unconnected-(J4-Pad2)")
+  (footprint "Display_local:Waveshare_EPD_1in9" (layer "F.Cu")
+    (at 31 80.25)
+    (descr "Waveshare EPD_1in9 Segmented e-Paper Display")
+    (tags "EPD, e-Paper, 1.9in, Waveshare")
+    (property "Manufacturer URL" "https://www.waveshare.com/wiki/1.9inch_Segment_e-Paper_Module")
+    (property "Sheetfile" "EPD_1in9.kicad_sch")
+    (property "Sheetname" "")
+    (fp_text reference "Disp1" (at 3 -48.25 unlocked) (layer "F.Fab")
+      (effects (font (size 1 1) (thickness 0.15)))
+    )
+    (fp_text value "Waveshare_EPD_1in9" (at 17 -25.5 unlocked) (layer "F.Fab")
+      (effects (font (size 1 1) (thickness 0.15)))
+    )
+    (fp_text user "${REFERENCE}" (at 17 -24 unlocked) (layer "F.Fab") hide
+      (effects (font (size 1 1) (thickness 0.15)))
+    )
+    (fp_line (start 12.3 -7.85) (end 12.3 -3.35) (layer "B.Fab") (width 0.1))
+    (fp_line (start 20.2 0.75) (end 20.2 -2.85) (layer "B.Fab") (width 0.1))
+    (fp_line (start 9.8 -3.35) (end 9.8 -7.85) (layer "B.Fab") (width 0.1))
+    (fp_line (start 15.8 -7.85) (end 15.8 -3.35) (layer "B.Fab") (width 0.1))
+    (fp_line (start 9.8 -7.85) (end 24.8 -7.85) (layer "B.Fab") (width 0.1))
+    (fp_line (start 25.8 0.75) (end 25.8 -6.85) (layer "B.Fab") (width 0.1))
+    (fp_line (start 19.7 -3.35) (end 9.8 -3.35) (layer "B.Fab") (width 0.1))
+    (fp_arc (start 19.7 -3.35) (mid 20.053553 -3.203553) (end 20.2 -2.85) (layer "B.Fab") (width 0.1))
+    (fp_arc (start 24.8 -7.85) (mid 25.507107 -7.557107) (end 25.8 -6.85) (layer "B.Fab") (width 0.1))
+    (fp_line (start 32 -49.5) (end 0 -49.5) (layer "F.Fab") (width 0.1))
+    (fp_line (start 20.2 0.75) (end 25.8 0.75) (layer "F.Fab") (width 0.1))
+    (fp_line (start 20.2 0) (end 20.2 0.75) (layer "F.Fab") (width 0.1))
+    (fp_line (start 0 -49.5) (end 0 0) (layer "F.Fab") (width 0.1))
+    (fp_line (start 25.8 0.75) (end 25.8 0) (layer "F.Fab") (width 0.1))
+    (fp_line (start 0 0) (end 32 0) (layer "F.Fab") (width 0.1))
+    (fp_line (start 32 0) (end 32 -49.5) (layer "F.Fab") (width 0.1))
+  )
   (footprint "Resistor_SMD:R_1206_3216Metric_Pad1.30x1.75mm_HandSolder" (layer "B.Cu")
     (at 45 57 -90)
@@
   (gr_line (start 63 81) (end 58.1 81) (layer "Edge.Cuts") (width 0.1))
   (gr_arc (start 31 81) (mid 30.292893 80.707107) (end 30 80) (layer "Edge.Cuts") (width 0.1))
-  (gr_line (start 56.8 81) (end 51.2 81) (layer "B.Fab") (width 0.1))
-  (gr_arc (start 50.7 76.9) (mid 51.053553 77.046447) (end 51.2 77.4) (layer "B.Fab") (width 0.1))
-  (gr_line (start 56.8 81) (end 56.8 73.4) (layer "B.Fab") (width 0.1))
-  (gr_arc (start 55.8 72.4) (mid 56.507107 72.692893) (end 56.8 73.4) (layer "B.Fab") (width 0.1))
   (gr_line (start 40.8 76.9) (end 40.8 72.4) (layer "B.Fab") (width 0.1))
-  (gr_line (start 43.3 72.4) (end 43.3 76.9) (layer "B.Fab") (width 0.1))
-  (gr_line (start 40.8 72.4) (end 55.8 72.4) (layer "B.Fab") (width 0.1))
-  (gr_line (start 51.2 81) (end 51.2 77.4) (layer "B.Fab") (width 0.1))
-  (gr_line (start 50.7 76.9) (end 40.8 76.9) (layer "B.Fab") (width 0.1))
-  (gr_line (start 46.8 72.4) (end 46.8 76.9) (layer "B.Fab") (width 0.1))
-  (gr_line (start 31 30.75) (end 31 80.25) (layer "F.Fab") (width 0.1))
-  (gr_line (start 56.8 81) (end 56.8 80.25) (layer "F.Fab") (width 0.1))
-  (gr_line (start 51.2 80.25) (end 51.2 81) (layer "F.Fab") (width 0.1))
-  (gr_line (start 51.2 81) (end 56.8 81) (layer "F.Fab") (width 0.1))
-  (gr_line (start 63 30.75) (end 31 30.75) (layer "F.Fab") (width 0.1))
-  (gr_line (start 31 80.25) (end 63 80.25) (layer "F.Fab") (width 0.1))
-  (gr_line (start 63 80.25) (end 63 30.75) (layer "F.Fab") (width 0.1))
   (gr_line (start 47 82) (end 47 29) (layer "F.Fab") (width 0.1))
+  (gr_text "Chris Baker 2023" (at 62 73 90) (layer "B.SilkS")
+    (effects (font (size 1 1) (thickness 0.15)) (justify mirror))
+  )
   (dimension (type aligned) (layer "F.Fab")
     (pts (xy 30 79.5) (xy 64 79.5))
