File: kicad/EPD_1in9/EPD_1in9.kicad_pcb (KiCad board)
At the start: 2 copper layers, 34 x 51 mm, 11 parts, among them J1 Conn_01x02, J2 Conn_01x08, J3 Conn_01x08, J4 Conn_01x08

Commit message: EPD_1in9: Add 3D-model for CF3527S connector
IGES model downloaded from:
https://www.cvilux.com/uploads/3d/101/681/CF35082D0RM_NH.zip

Cleaned up colors in FreeCAD and exported as VRML.

Also updated some of the footprint properties and renamed
from CF35 to CF3527S.
Parts:
- J4: footprint Connector:CivLux_CF35_1x08-1MP_P0.50mm_Horizontal -> Connector_local:CivLux_CF3527S_1x08-1MP_P0.50mm_Horizontal
Other:
- board text added: "EPD_1in9 Rev B"
Changed lines of the file:
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@@
     )
   )
-  (footprint "Connector:CivLux_CF35_1x08-1MP_P0.50mm_Horizontal" (layer "B.Cu")
+  (footprint "Connector_local:CivLux_CF3527S_1x08-1MP_P0.50mm_Horizontal" (layer "B.Cu")
     (at 41.7 74.65 -90)
-    (descr "CivLux CF35, FFC/FPC connector, CF3508WD, 8 Pins per row")
-    (tags "connector CivLux CF35 horizontal")
+    (descr "CivLux CF3527S (RM Type), FFC/FPC connector, CF3508WD, 8 Pins per row")
+    (tags "connector CivLux CF3527S horizontal")
     (property "Sheetfile" "EPD_1in9.kicad_sch")
     (property "Sheetname" "")
     (attr smd)
-    (fp_text reference "J4" (at 0 3.2 90) (layer "B.SilkS")
+    (fp_text reference "J4" (at 0 3.9 90) (layer "B.SilkS")
       (effects (font (size 1 1) (thickness 0.15)) (justify mirror))
     )
-    (fp_text value "Conn_01x08" (at 4.35 -1.3 180) (layer "B.Fab")
+    (fp_text value "Conn_01x08" (at 0 -5.4 90) (layer "B.Fab")
+      (effects (font (size 1 1) (thickness 0.15)) (justify mirror))
+    )
+    (fp_text user "https://www.cvilux.com/uploads/spec/101/681/SPCF053.pdf" (at 0 0 90) (layer "B.Fab") hide
+      (effects (font (size 1 1) (thickness 0.15)) (justify mirror))
+    )
+    (fp_text user "https://www.cvilux.com/uploads/drawings/101/681/CF3527S.pdf" (at 0 0 90) (layer "B.Fab") hide
+      (effects (font (size 1 1) (thickness 0.15)) (justify mirror))
+    )
+    (fp_text user "https://www.cvilux.com/uploads/3d/101/681/CF35082D0RM_NH.zip" (at 0 0 90) (layer "B.Fab") hide
       (effects (font (size 1 1) (thickness 0.15)) (justify mirror))
     )
@@
       (effects (font (size 1 1) (thickness 0.15)) (justify mirror))
     )
+    (fp_line (start -2.15 1.6) (end -3.55 1.6) (layer "B.SilkS") (width 0.12))
+    (fp_line (start 3.55 -2.8) (end 3.55 -0.3) (layer "B.SilkS") (width 0.12))
+    (fp_line (start -3.55 1.6) (end -3.55 0.3) (layer "B.SilkS") (width 0.12))
+    (fp_line (start 3.55 1.6) (end 3.55 0.3) (layer "B.SilkS") (width 0.12))
     (fp_line (start 2.15 1.6) (end 3.55 1.6) (layer "B.SilkS") (width 0.12))
+    (fp_line (start -3.55 -2.8) (end 3.55 -2.8) (layer "B.SilkS") (width 0.12))
     (fp_line (start -3.55 -0.3) (end -3.55 -2.8) (layer "B.SilkS") (width 0.12))
-    (fp_line (start 3.55 1.6) (end 3.55 0.3) (layer "B.SilkS") (width 0.12))
-    (fp_line (start 3.55 -2.8) (end 3.55 -0.3) (layer "B.SilkS") (width 0.12))
-    (fp_line (start -2.15 1.6) (end -3.55 1.6) (layer "B.SilkS") (width 0.12))
-    (fp_line (start -3.55 -2.8) (end 3.55 -2.8) (layer "B.SilkS") (width 0.12))
-    (fp_line (start -3.55 1.6) (end -3.55 0.3) (layer "B.SilkS") (width 0.12))
     (fp_line (start -2.15 1.6) (end -2.15 2.4) (layer "B.SilkS") (width 0.12))
+    (fp_line (start -4 -6) (end 4 -6) (layer "B.CrtYd") (width 0.05))
+    (fp_line (start 4 -6) (end 4 4) (layer "B.CrtYd") (width 0.05))
+    (fp_line (start 4 4) (end -4 4) (layer "B.CrtYd") (width 0.05))
     (fp_line (start -4 4) (end -4 -6) (layer "B.CrtYd") (width 0.05))
-    (fp_line (start 4 4) (end -4 4) (layer "B.CrtYd") (width 0.05))
-    (fp_line (start 4 -6) (end 4 4) (layer "B.CrtYd") (width 0.05))
-    (fp_line (start -4 -6) (end 4 -6) (layer "B.CrtYd") (width 0.05))
+    (fp_line (start 0 0.9) (end -2.95 0.9) (layer "B.Fab") (width 0.1))
+    (fp_line (start -2.6 -1.1) (end -2.6 -2.5) (layer "B.Fab") (width 0.1))
     (fp_line (start 2.95 -1.1) (end 2.6 -1.1) (layer "B.Fab") (width 0.1))
-    (fp_line (start -2.6 -1.1) (end -2.6 -2.5) (layer "B.Fab") (width 0.1))
+    (fp_line (start 2.6 -2.5) (end 0 -2.5) (layer "B.Fab") (width 0.1))
+    (fp_line (start 2.6 -1.1) (end 2.6 -2.5) (layer "B.Fab") (width 0.1))
+    (fp_line (start -2.95 -1.1) (end -2.6 -1.1) (layer "B.Fab") (width 0.1))
+    (fp_line (start 2.95 0.9) (end 2.95 -1.1) (layer "B.Fab") (width 0.1))
     (fp_line (start 0 0.9) (end 2.95 0.9) (layer "B.Fab") (width 0.1))
-    (fp_line (start 0 0.9) (end -2.95 0.9) (layer "B.Fab") (width 0.1))
-    (fp_line (start 2.6 -1.1) (end 2.6 -2.5) (layer "B.Fab") (width 0.1))
+    (fp_line (start -2.95 0.9) (end -2.95 -1.1) (layer "B.Fab") (width 0.1))
     (fp_line (start -2.6 -2.5) (end 0 -2.5) (layer "B.Fab") (width 0.1))
-    (fp_line (start -2.95 -1.1) (end -2.6 -1.1) (layer "B.Fab") (width 0.1))
-    (fp_line (start -2.95 0.9) (end -2.95 -1.1) (layer "B.Fab") (width 0.1))
-    (fp_line (start 2.6 -2.5) (end 0 -2.5) (layer "B.Fab") (width 0.1))
-    (fp_line (start 2.95 0.9) (end 2.95 -1.1) (layer "B.Fab") (width 0.1))
     (pad "1" smd roundrect (at -1.75 1.25 270) (size 0.3 1.3) (layers "B.Cu" "B.Paste" "B.Mask") (roundrect_rratio 0.25)
       (net 3 "/HV") (pinfunction "Pin_1") (pintype "passive") (solder_paste_margin -0.07))
@@
     (pad "MP" smd roundrect (at -2.85 -1.7 270) (size 0.5 1.4) (layers "B.Cu" "B.Paste" "B.Mask") (roundrect_rratio 0.25)
       (solder_paste_margin -0.08))
-    (model "${KICAD6_3DMODEL_DIR}/Connector_FFC-FPC.3dshapes/Hirose_FH12-8S-0.5SH_1x08-1MP_P0.50mm_Horizontal.wrl"
-      (offset (xyz 0 0 0))
-      (scale (xyz 1 1 1))
+    (model "${KIPRJMOD}/CF35082D0RM_NH.wrl"
+      (offset (xyz 0 -1.5 0))
+      (scale (xyz 0.3937 0.3937 0.3937))
       (rotate (xyz 0 0 0))
     )
@@
   (gr_line (start 40.8 76.9) (end 40.8 72.4) (layer "B.Fab") (width 0.1))
   (gr_line (start 47 82) (end 47 29) (layer "F.Fab") (width 0.1))
+  (gr_text "EPD_1in9 Rev B" (at 62 56 90) (layer "B.SilkS")
+    (effects (font (size 1 1) (thickness 0.15)) (justify mirror))
+  )
   (gr_text "Chris Baker 2023" (at 62 73 90) (layer "B.SilkS")
     (effects (font (size 1 1) (thickness 0.15)) (justify mirror))
